Commit message: Update hokuyo_mount.urdf.xacro
added support for v4s

File: bwi_ros2_common/segbot_description/urdf/mounts/hokuyo_mount.urdf.xacro (robot description, xacro)
@@ -16,11 +16,11 @@
     </xacro:hokuyo_laser>
   </xacro:macro>
-  <!-- <xacro:macro name="hokuyo_mount" params="name parent *origin length ros_topic update_rate min_angle max_angle rrange">
+  <xacro:macro name="hokuyo_mount" params="name parent *origin length ros_topic update_rate min_angle max_angle hmrange">
     <xacro:beam_8020 name="${name}_sensor_beam" parent="${parent}" length="${length}">
       <xacro:insert_block name="origin" />
     </xacro:beam_8020>
-    <xacro:hokuyo_mount_without_beam name="${name}" parent="${name}_sensor_beam" ros_topic="${ros_topic}" update_rate="${update_rate}" min_angle="${min_angle}" max_angle="${max_angle}" lrange="${rrange}">
+    <xacro:hokuyo_mount_without_beam name="${name}" parent="${name}_sensor_beam" ros_topic="${ros_topic}" update_rate="${update_rate}" min_angle="${min_angle}" max_angle="${max_angle}" lrange="${hmrange}">
       <origin xyz="${0.5*INCH_TO_M} ${0.75*INCH_TO_M} ${length/2}" rpy="${M_PI/2} 0 ${M_PI/2}" />
     </xacro:hokuyo_mount_without_beam>
-  </xacro:macro> -->
+  </xacro:macro>
 </root>
